File: TwirrePCB/Shield.sch (EAGLE design)
At the start: 38 parts, among them Q1 BSS138, Q2 BSS138, T2 BC847, U1 ARDUINO-MEGAPRO

Commit message: Add various components to library
Parts:
- removed SV10, SV7, SV8, SV9: (no value), con-lstb:MA04-1
- removed SV11: LIPO, con-lsta:FE05-1
- added LED3: (no value), led:LEDSML0805
- added R21, R6, R7: 100, resistor:R-EU_R0805
- added R22: (no value), resistor:R-EU_R0805
- added S1: (no value), switch-omron:10-XX
- added U$1: RGB5MMRGB5MM, Arduino-Boards:RGB5MMRGB5MM
- added U$10, U$11, U$2, U$3, U$4, U$5, U$6, U$7, U$8, U$9: JST-4, Arduino-Boards:JST-4
- added U$12, U$13: LIDAR, Arduino-Boards:JST-5
- added U$14, U$15: JST-3, Arduino-Boards:JST-3
- added U$16: JST-2, Arduino-Boards:JST-2
- LED2: device led:LED5MM -> led:LEDSML0805
- SV2, SV3: device con-lstb:MA04-1 -> con-lsta:FE08-1
- SV4, SV5, SV6: device con-lstb:MA04-1 -> con-lstb:MA03-2
Connections:
- new net N$20: R7.2, U1.46
- new net N$21: R20.1, U$1.P3
- new net N$22: R6.1, U$1.P2
- new net N$23: R7.1, U$1.P1
- new net N$24: SV2.2, U1.45
- new net N$25: SV5.6, U1.35
- new net N$26: SV5.5, U1.33
- new net N$27: SV4.6, U1.31
- new net N$28: SV6.6, U1.39
- new net N$29: SV6.5, U1.37
- new net N$30: LED2.A, R21.2
- new net N$31: SV4.5, U1.29
- new net N$32: R21.1, U1.23
- new net N$33: LED3.A, R22.2
- new net N$34: S1.S, S1.S1, U1.RESET
- new net N$35: U$16.2, U1.VIN
- net +3V3: now also SV2.7, U$10.4, U$14.2, U$15.2, U$2.4, U$3.4, U$4.4, U$8.4, U$9.4, U1.3.3V; no longer SV10.1, SV2.1, SV3.1, SV4.1, SV8.1, SV9.1
- net +5V: now also R22.1, SV4.1, SV4.2, SV5.2, SV6.2, U$11.4, U$12.5, U$14.3, U$15.3, U$5.4, U$6.4, U$7.4, U1.5V@0, U1.5V@1, U1.5V@2; no longer SV7.1
- net GND: now also LED3.C, S1.P, S1.P1, SV2.8, SV4.3, SV5.3, SV6.3, U$1.C, U$10.1, U$11.1, U$12.1, U$13.1, U$14.1, U$15.1, U$16.1, U$2.1, U$3.1, U$4.1, U$5.1, U$6.1, U$7.1, U$8.1, U$9.1; no longer SV10.4, SV11.1, SV2.4, SV3.4, SV7.4, SV8.4, SV9.4
- net N$10: now also U$13.3; no longer SV11.3
- net N$11: now also U$13.4; no longer SV11.4
- net N$12: now also U$13.5; no longer SV11.5
- net N$15: now also R6.2, U1.47; no longer LED2.A, R20.1
- net N$7: now also U$13.2; no longer SV11.2
- net SCL_HS: now also U$10.2, U$8.2, U$9.2, U1.21(SCL); no longer SV10.3, SV8.3, SV9.3, U1.HS_SCL
- net SCL_LS: now also SV2.5, U$12.3, U$2.2, U$3.2, U$4.2, U1.HS_SCL; no longer SV2.3, SV3.3, SV4.3, U1.21(SCL)
- net SCL_LS_5: now also U$11.2, U$5.2, U$6.2, U$7.2; no longer SV5.3, SV6.3, SV7.3
- net SDA_HS: now also U$10.3, U$8.3, U$9.3, U1.20(SDA); no longer SV10.2, SV8.2, SV9.2, U1.HS_SDA
- net SDA_LS: now also SV2.6, U$12.4, U$2.3, U$3.3, U$4.3, U1.HS_SDA; no longer SV2.2, SV3.2, SV4.2, U1.20(SDA)
- net SDA_LS_5: now also U$11.3, U$5.3, U$6.3, U$7.3; no longer SV5.2, SV6.2, SV7.2
Other:
- note added: "Lidar"
- moved on the sheet: LED2, R20

Commit message: Add caps and lots of other stuff
Parts:
- removed SV1: PWM IN, con-lstb:MA06-1
- removed SV14: PWM OUT, con-lstb:MA05-1
- removed SV4, SV5, SV6: (no value), con-lstb:MA03-2
- added C1: 560uF, resistor:CPOL-EU153CLV-1010
- added C2: (no value), resistor:CPOL-EU153CLV-0605
- added U$17: JST-6, Arduino-Boards:JST-6
- added U$18: JST-5, Arduino-Boards:JST-5
- added U$19, U$20, U$21, U$22, U$23, U$24: SERVOHEADER, Arduino-Boards:SERVOHEADER
- R22: value (none) -> 220
Connections:
- removed net N$31: SV4.5, U1.29
- new net N$36: U$24.S, U1.29
- net +3V3: now also C2.+
- net +5V: now also C1.+, U$19.+, U$20.+, U$21.+, U$22.+, U$23.+, U$24.+; no longer SV4.1, SV4.2, SV5.1, SV5.2, SV6.1, SV6.2
- net GND: now also C1.-, C2.-, U$17.1, U$18.1, U$19.-, U$20.-, U$21.-, U$22.-, U$23.-, U$24.-; no longer SV1.1, SV14.1, SV4.3, SV4.4, SV5.3, SV5.4, SV6.3, SV6.4
- net N$13: now also U$17.6; no longer SV1.2
- net N$16: now also U$18.2; no longer SV14.5
- net N$17: now also U$18.3; no longer SV14.4
- net N$18: now also U$18.4; no longer SV14.3
- net N$19: now also U$18.5; no longer SV14.2
- net N$25: now also U$21.S; no longer SV5.6
- net N$26: now also U$22.S; no longer SV5.5
- net N$27: now also U$23.S; no longer SV4.6
- net N$28: now also U$19.S; no longer SV6.6
- net N$29: now also U$20.S; no longer SV6.5
- net N$5: now also U$17.5, U1.5; no longer SV1.6, U1.2
- net N$6: now also U$17.4, U1.4; no longer SV1.5, U1.3
- net N$8: now also U$17.3, U1.3; no longer SV1.4, U1.4
- net N$9: now also U$17.2, U1.2; no longer SV1.3, U1.5
Other:
- note added: "PWM IN"
- note added: "PWM OUT"
- moved on the sheet: LED2, LED3, R21, R22

Commit message: Move some parts and wires around, finished first revision
Parts:
- removed SV13: (no value), con-lstb:MA04-2
- added U$25: IDC-8WAY, Arduino-Boards:IDC-8WAY
- C2: value (none) -> 47uF
Connections:
- removed net SCL: SV13.8
- removed net SDA: SV13.7
- net GND: now also U$25.5; no longer SV13.5
- net SCL_LS: now also U$25.8
- net SDA_LS: now also U$25.7
- net SPI_CLK: now also U$25.4; no longer SV13.4
- net SPI_CS: now also U$25.1; no longer SV13.1
- net SPI_MISO: now also U$25.3; no longer SV13.3
- net SPI_MOSI: now also U$25.2; no longer SV13.2
- net SPI_VIN: now also U$25.6; no longer SV13.6
Changed lines of the file:
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@@
 <part name="GND11" library="supply1" deviceset="GND" device=""/>
 <part name="R20" library="resistor" deviceset="R-EU_" device="R0805" value="100"/>
-<part name="SV13" library="con-lstb" deviceset="MA04-2" device=""/>
 <part name="GND13" library="supply1" deviceset="GND" device=""/>
 <part name="GND14" library="supply1" deviceset="GND" device=""/>
@@
 <part name="P+10" library="supply1" deviceset="+5V" device=""/>
 <part name="GND20" library="supply1" deviceset="GND" device=""/>
-<part name="C2" library="resistor" deviceset="CPOL-EU" device="153CLV-0605"/>
+<part name="C2" library="resistor" deviceset="CPOL-EU" device="153CLV-0605" value="47uF"/>
 <part name="+3V10" library="supply1" deviceset="+3V3" device=""/>
+<part name="U$25" library="Arduino-Boards" deviceset="IDC-8WAY" device=""/>
 </parts>
 <sheets>
@@
 <attribute name="VALUE" x="92.71" y="33.782" size="1.778" layer="96" rot="R180"/>
 </instance>
-<instance part="SV13" gate="G$1" x="269.24" y="30.48" rot="MR180"/>
 <instance part="GND13" gate="1" x="-2.54" y="66.04"/>
 <instance part="GND14" gate="1" x="-2.54" y="38.1"/>
@@
 <instance part="C2" gate="G$1" x="55.88" y="180.34"/>
 <instance part="+3V10" gate="G$1" x="55.88" y="187.96"/>
+<instance part="U$25" gate="G$1" x="274.32" y="30.48" rot="MR0"/>
 </instances>
 <busses>
@@
 <net name="SPI_CS" class="0">
 <segment>
-<junction x="287.02" y="35.56"/>
-<pinref part="SV13" gate="G$1" pin="1"/>
-<wire x1="287.02" y1="35.56" x2="276.86" y2="35.56" width="0.1524" layer="91"/>
-<label x="279.4" y="35.56" size="1.778" layer="95"/>
+<junction x="304.8" y="35.56"/>
+<wire x1="304.8" y1="35.56" x2="287.02" y2="35.56" width="0.1524" layer="91"/>
+<label x="297.18" y="35.56" size="1.778" layer="95"/>
+<pinref part="U$25" gate="G$1" pin="1"/>
 </segment>
 <segment>
@@
 <segment>
 <junction x="248.92" y="35.56"/>
-<pinref part="SV13" gate="G$1" pin="2"/>
 <wire x1="248.92" y1="35.56" x2="261.62" y2="35.56" width="0.1524" layer="91"/>
 <label x="248.92" y="35.56" size="1.778" layer="95"/>
+<pinref part="U$25" gate="G$1" pin="2"/>
 </segment>
 <segment>
@@
 <net name="SPI_MISO" class="0">
 <segment>
-<junction x="287.02" y="33.02"/>
-<pinref part="SV13" gate="G$1" pin="3"/>
-<wire x1="287.02" y1="33.02" x2="276.86" y2="33.02" width="0.1524" layer="91"/>
-<label x="279.4" y="33.02" size="1.778" layer="95"/>
+<junction x="304.8" y="33.02"/>
+<wire x1="304.8" y1="33.02" x2="287.02" y2="33.02" width="0.1524" layer="91"/>
+<label x="297.18" y="33.02" size="1.778" layer="95"/>
+<pinref part="U$25" gate="G$1" pin="3"/>
 </segment>
 <segment>
@@
 <segment>
 <junction x="248.92" y="33.02"/>
-<pinref part="SV13" gate="G$1" pin="4"/>
 <wire x1="248.92" y1="33.02" x2="261.62" y2="33.02" width="0.1524" layer="91"/>
 <label x="248.92" y="33.02" size="1.778" layer="95"/>
+<pinref part="U$25" gate="G$1" pin="4"/>
 </segment>
 <segment>
@@
 <net name="GND" class="0">
 <segment>
-<junction x="287.02" y="30.48"/>
-<pinref part="SV13" gate="G$1" pin="5"/>
-<wire x1="287.02" y1="30.48" x2="276.86" y2="30.48" width="0.1524" layer="91"/>
-<label x="279.4" y="30.48" size="1.778" layer="95"/>
+<junction x="304.8" y="30.48"/>
+<wire x1="304.8" y1="30.48" x2="287.02" y2="30.48" width="0.1524" layer="91"/>
+<label x="297.18" y="30.48" size="1.778" layer="95"/>
+<pinref part="U$25" gate="G$1" pin="5"/>
 </segment>
 <segment>
@@
 <wire x1="233.68" y1="25.4" x2="233.68" y2="30.48" width="0.1524" layer="91"/>
 <junction x="233.68" y="30.48"/>
-<pinref part="SV13" gate="G$1" pin="6"/>
 <wire x1="233.68" y1="30.48" x2="261.62" y2="30.48" width="0.1524" layer="91"/>
-</segment>
-</net>
-<net name="SDA" class="0">
-<segment>
-<junction x="287.02" y="27.94"/>
-<pinref part="SV13" gate="G$1" pin="7"/>
-<wire x1="287.02" y1="27.94" x2="276.86" y2="27.94" width="0.1524" layer="91"/>
-<label x="279.4" y="27.94" size="1.778" layer="95"/>
-</segment>
-</net>
-<net name="SCL" class="0">
-<segment>
-<junction x="248.92" y="27.94"/>
-<wire x1="248.92" y1="27.94" x2="261.62" y2="27.94" width="0.1524" layer="91"/>
-<pinref part="SV13" gate="G$1" pin="8"/>
-<label x="248.92" y="27.94" size="1.778" layer="95"/>
+<pinref part="U$25" gate="G$1" pin="6"/>
 </segment>
 </net>
@@
 <wire x1="154.94" y1="88.9" x2="154.94" y2="81.28" width="0.1524" layer="91"/>
 </segment>
+<segment>
+<junction x="248.92" y="27.94"/>
+<wire x1="248.92" y1="27.94" x2="261.62" y2="27.94" width="0.1524" layer="91"/>
+<label x="248.92" y="27.94" size="1.778" layer="95"/>
+<pinref part="U$25" gate="G$1" pin="8"/>
+</segment>
 </net>
 <net name="SDA_LS" class="0">
@@
 <wire x1="157.48" y1="88.9" x2="157.48" y2="81.28" width="0.1524" layer="91"/>
 </segment>
-</net>
+<segment>
+<junction x="304.8" y="27.94"/>
+<wire x1="304.8" y1="27.94" x2="287.02" y2="27.94" width="0.1524" layer="91"/>
+<label x="297.18" y="27.94" size="1.778" layer="95"/>
+<pinref part="U$25" gate="G$1" pin="7"/>
+</segment>
+</net>

Commit message: Minor trace modifications
Connections:
- net SCL_HS: now also U$12.3
- net SCL_LS: no longer U$12.3
- net SDA_HS: now also U$12.4
- net SDA_LS: no longer U$12.4
Changed lines of the file:
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@@
-</segment>
-<segment>
-<pinref part="U$12" gate="G$1" pin="3"/>
-<wire x1="180.34" y1="127" x2="162.56" y2="127" width="0.1524" layer="91"/>
-<label x="154.94" y="127" size="1.778" layer="95"/>
 </segment>
 <segment>
@@
 <wire x1="73.66" y1="22.86" x2="88.9" y2="22.86" width="0.1524" layer="91"/>
 <label x="83.82" y="22.86" size="1.778" layer="95"/>
-</segment>
-<segment>
-<pinref part="U$12" gate="G$1" pin="4"/>
-<wire x1="180.34" y1="129.54" x2="162.56" y2="129.54" width="0.1524" layer="91"/>
-<label x="154.94" y="129.54" size="1.778" layer="95"/>
 </segment>
 <segment>
@@
 <label x="86.36" y="109.22" size="1.778" layer="95"/>
 </segment>
+<segment>
+<pinref part="U$12" gate="G$1" pin="4"/>
+<wire x1="180.34" y1="129.54" x2="162.56" y2="129.54" width="0.1524" layer="91"/>
+<label x="154.94" y="129.54" size="1.778" layer="95"/>
+</segment>
 </net>
 <net name="SCL_HS" class="0">
@@
 <label x="86.36" y="106.68" size="1.778" layer="95"/>
 </segment>
-</net>
+<segment>
+<pinref part="U$12" gate="G$1" pin="3"/>
+<wire x1="180.34" y1="127" x2="162.56" y2="127" width="0.1524" layer="91"/>
+<label x="154.94" y="127" size="1.778" layer="95"/>
+</segment>
+</net>

Commit message: Increase LED Resistor values
Parts:
- R20, R21, R6, R7: value 100 -> 220
Changed lines of the file:
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@@
 <part name="GND10" library="supply1" deviceset="GND" device=""/>
 <part name="GND11" library="supply1" deviceset="GND" device=""/>
-<part name="R20" library="resistor" deviceset="R-EU_" device="R0805" value="100"/>
+<part name="R20" library="resistor" deviceset="R-EU_" device="R0805" value="220"/>
 <part name="GND13" library="supply1" deviceset="GND" device=""/>
 <part name="GND14" library="supply1" deviceset="GND" device=""/>
 <part name="+3V6" library="supply1" deviceset="+3V3" device=""/>
 <part name="P+4" library="supply1" deviceset="+5V" device=""/>
-<part name="R6" library="resistor" deviceset="R-EU_" device="R0805" value="100"/>
-<part name="R7" library="resistor" deviceset="R-EU_" device="R0805" value="100"/>
+<part name="R6" library="resistor" deviceset="R-EU_" device="R0805" value="220"/>
+<part name="R7" library="resistor" deviceset="R-EU_" device="R0805" value="220"/>
 <part name="GND12" library="supply1" deviceset="GND" device=""/>
 <part name="U$1" library="Arduino-Boards" deviceset="RGB5MM" device="RGB5MM"/>
@@
 <part name="P+7" library="supply1" deviceset="+5V" device=""/>
 <part name="P+8" library="supply1" deviceset="+5V" device=""/>
-<part name="R21" library="resistor" deviceset="R-EU_" device="R0805" value="100"/>
+<part name="R21" library="resistor" deviceset="R-EU_" device="R0805" value="220"/>
 <part name="LED2" library="led" deviceset="LED" device="SML0805"/>
 <part name="R22" library="resistor" deviceset="R-EU_" device="R0805" value="220"/>

Commit message: Change Transistors for FMMT491A and FMMT591A
Parts:
- removed T1: (no value), transistor:BC857A-PNP-SOT23-BEC
- removed T2: BC847, transistor:BC847
- added T3: FMMT591A, transistor:-PNP-SOT23-BCE
- added T4: FMMT491A, transistor:BC808-NPN-SOT23-BEC
Connections:
- net +3V3: now also T3.E; no longer T1.E
- net GND: now also T4.E; no longer T2.E
- net N$1: now also T3.B; no longer T1.B
- net N$2: now also T4.C; no longer T2.C
- net N$3: now also T4.B; no longer T2.B
- net SPI_VIN: now also T3.C; no longer T1.C
Changed lines of the file:
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@@
 <part name="GND1" library="supply1" deviceset="GND" device=""/>
 <part name="GND2" library="supply1" deviceset="GND" device=""/>
-<part name="T1" library="transistor" deviceset="*-PNP-" device="SOT23-BEC" technology="BC857A"/>
-<part name="T2" library="transistor" deviceset="BC847" device=""/>
 <part name="R1" library="resistor" deviceset="R-EU_" device="R0805" value="10k"/>
 <part name="R2" library="resistor" deviceset="R-EU_" device="R0805" value="1k"/>
@@
 <part name="+3V10" library="supply1" deviceset="+3V3" device=""/>
 <part name="U$25" library="Arduino-Boards" deviceset="IDC-8WAY" device=""/>
+<part name="T3" library="transistor" deviceset="*-PNP-" device="SOT23-BCE" value="FMMT591A "/>
+<part name="T4" library="transistor" deviceset="*-NPN-" device="SOT23-BEC" technology="BC808" value="FMMT491A "/>
 </parts>
 <sheets>
@@
 <text x="200.66" y="195.58" size="1.778" layer="91">+</text>
 <text x="200.66" y="187.96" size="1.778" layer="91">-</text>
-<text x="-149.86" y="86.36" size="1.778" layer="91" rot="R90">MAX 4.2V PER CELL</text>
-<text x="-152.4" y="86.36" size="1.778" layer="91" rot="R90">16.8V TOTAL</text>
+<text x="-147.32" y="86.36" size="1.778" layer="91" rot="R90">MAX 4.2V PER CELL</text>
+<text x="-149.86" y="86.36" size="1.778" layer="91" rot="R90">16.8V TOTAL</text>
 <text x="-111.76" y="91.44" size="1.778" layer="91">4.2V</text>
 <text x="-93.98" y="93.98" size="1.778" layer="91">8.4V</text>
@@
 <instance part="GND1" gate="1" x="22.86" y="22.86"/>
 <instance part="GND2" gate="1" x="81.28" y="5.08"/>
-<instance part="T1" gate="G$1" x="231.14" y="38.1"/>
-<instance part="T2" gate="G$1" x="223.52" y="17.78"/>
 <instance part="R1" gate="G$1" x="226.06" y="45.72" rot="R90"/>
 <instance part="R2" gate="G$1" x="226.06" y="30.48" rot="R90"/>
@@
 <instance part="+3V10" gate="G$1" x="55.88" y="187.96"/>
 <instance part="U$25" gate="G$1" x="274.32" y="30.48" rot="MR0"/>
+<instance part="T3" gate="G$1" x="231.14" y="38.1"/>
+<instance part="T4" gate="G$1" x="223.52" y="17.78"/>
 </instances>
 <busses>
@@
 <wire x1="218.44" y1="5.08" x2="218.44" y2="2.54" width="0.1524" layer="91"/>
 <wire x1="218.44" y1="2.54" x2="220.98" y2="2.54" width="0.1524" layer="91"/>
-<pinref part="T2" gate="G$1" pin="E"/>
 <wire x1="220.98" y1="2.54" x2="226.06" y2="2.54" width="0.1524" layer="91"/>
 <wire x1="226.06" y1="2.54" x2="226.06" y2="12.7" width="0.1524" layer="91"/>
@@
 <wire x1="233.68" y1="2.54" x2="233.68" y2="5.08" width="0.1524" layer="91"/>
 <junction x="226.06" y="2.54"/>
+<pinref part="T4" gate="G$1" pin="E"/>
 </segment>
 <segment>
@@
 <net name="SPI_VIN" class="0">
 <segment>
-<pinref part="T1" gate="G$1" pin="C"/>
 <wire x1="233.68" y1="33.02" x2="233.68" y2="30.48" width="0.1524" layer="91"/>
 <pinref part="R5" gate="G$1" pin="1"/>
@@
 <wire x1="233.68" y1="30.48" x2="261.62" y2="30.48" width="0.1524" layer="91"/>
 <pinref part="U$25" gate="G$1" pin="6"/>
+<pinref part="T3" gate="G$1" pin="C"/>
 </segment>
 </net>
@@
 <net name="N$1" class="0">
 <segment>
-<pinref part="T1" gate="G$1" pin="B"/>
 <wire x1="228.6" y1="38.1" x2="226.06" y2="38.1" width="0.1524" layer="91"/>
 <pinref part="R1" gate="G$1" pin="1"/>
@@
 <wire x1="226.06" y1="38.1" x2="226.06" y2="35.56" width="0.1524" layer="91"/>
 <junction x="226.06" y="38.1"/>
+<pinref part="T3" gate="G$1" pin="B"/>
 </segment>
 </net>
 <net name="N$2" class="0">
 <segment>
-<pinref part="T2" gate="G$1" pin="C"/>
 <pinref part="R2" gate="G$1" pin="1"/>
 <wire x1="226.06" y1="22.86" x2="226.06" y2="25.4" width="0.1524" layer="91"/>
+<pinref part="T4" gate="G$1" pin="C"/>
 </segment>
 </net>
@@
 <segment>
 <pinref part="R3" gate="G$1" pin="1"/>
-<pinref part="T2" gate="G$1" pin="B"/>
 <wire x1="215.9" y1="17.78" x2="218.44" y2="17.78" width="0.1524" layer="91"/>
 <pinref part="R4" gate="G$1" pin="1"/>
@@
 <wire x1="218.44" y1="15.24" x2="218.44" y2="17.78" width="0.1524" layer="91"/>
 <junction x="218.44" y="17.78"/>
+<pinref part="T4" gate="G$1" pin="B"/>
 </segment>
 </net>
@@
 </segment>
 <segment>
-<pinref part="T1" gate="G$1" pin="E"/>
 <wire x1="233.68" y1="43.18" x2="233.68" y2="55.88" width="0.1524" layer="91"/>
 <wire x1="233.68" y1="55.88" x2="226.06" y2="55.88" width="0.1524" layer="91"/>
@@
 <junction x="226.06" y="55.88"/>
 <pinref part="+3V2" gate="G$1" pin="+3V3"/>
-</segment>
-<segment>
+<pinref part="T3" gate="G$1" pin="E"/>
+</segment>
+<segment>
